File: PCBs/CustomKeyboard_Beryl/CustomKeyboard.kicad_sch (KiCad schematic)
At the start: 4 parts, among them J1 S2B-PH-K-SLFSN, SW1 SW_Push, SW2 SW_DPDT_x2, U2 nice_nano

Commit message: Completed Build!
Connections:
- net GND: now also J1.1; no longer J1.2
- net at SW2.1 (A): now also J1.2; no longer J1.1
Changed lines of the file:
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@@
 	(wire
 		(pts
-			(xy 198.12 67.31) (xy 198.12 59.69)
+			(xy 200.66 67.31) (xy 200.66 59.69)
 		)
 		(stroke
@@
 	(wire
 		(pts
-			(xy 207.01 81.28) (xy 201.93 81.28)
+			(xy 200.66 67.31) (xy 204.47 67.31)
 		)
 		(stroke
@@
 	(wire
 		(pts
-			(xy 204.47 67.31) (xy 198.12 67.31)
+			(xy 207.01 81.28) (xy 201.93 81.28)
 		)
 		(stroke
@@
 				(justify right)
 				(hide yes)
-			)
-		)
-	)
-	(symbol
-		(lib_id "power:GND")
-		(at 200.66 59.69 0)
-		(unit 1)
-		(exclude_from_sim no)
-		(in_bom yes)
-		(on_board yes)
-		(dnp no)
-		(fields_autoplaced yes)
-		(property "Reference" "#PWR05"
-			(at 200.66 66.04 0)
-			(effects
-				(font
-					(size 1.27 1.27)
-				)
-				(hide yes)
-			)
-		)
-		(property "Value" "GND"
-			(at 200.66 64.77 0)
-			(effects
-				(font
-					(size 1.27 1.27)
-				)
-			)
-		)
-		(property "Footprint" ""
-			(at 200.66 59.69 0)
-			(effects
-				(font
-					(size 1.27 1.27)
-				)
-				(hide yes)
-			)
-		)
-		(property "Datasheet" ""
-			(at 200.66 59.69 0)
-			(effects
-				(font
-					(size 1.27 1.27)
-				)
-				(hide yes)
-			)
-		)
-		(property "Description" "Power symbol creates a global label with name \"GND\" , ground"
-			(at 200.66 59.69 0)
-			(effects
-				(font
-					(size 1.27 1.27)
-				)
-				(hide yes)
-			)
-		)
-		(pin "1"
-		)
-		(instances
-			(project "CustomKeyboard"
-				(path "/e015e616-37c3-4f95-aa49-76389b12ce2e"
-					(reference "#PWR05")
-					(unit 1)
-				)
 			)
 		)
@@
 					(unit 1)
 				)
+			)
+		)
+	)
+	(symbol
+		(lib_id "power:GND")
+		(at 198.12 59.69 0)
+		(unit 1)
+		(exclude_from_sim no)
+		(in_bom yes)
+		(on_board yes)
+		(dnp no)
+		(fields_autoplaced yes)
+		(property "Reference" "#PWR05"
+			(at 198.12 66.04 0)
+			(effects
+				(font
+					(size 1.27 1.27)
+				)
+				(hide yes)
+			)
+		)
+		(property "Value" "GND"
+			(at 198.12 64.77 0)
+			(effects
+				(font
+					(size 1.27 1.27)
+				)
+			)
+		)
+		(property "Footprint" ""
+			(at 198.12 59.69 0)
+			(effects
+				(font
+					(size 1.27 1.27)
+				)
+				(hide yes)
+			)
+		)
+		(property "Datasheet" ""
+			(at 198.12 59.69 0)
+			(effects
+				(font
+					(size 1.27 1.27)
+				)
+				(hide yes)
+			)
+		)
+		(property "Description" "Power symbol creates a global label with name \"GND\" , ground"
+			(at 198.12 59.69 0)
+			(effects
+				(font
+					(size 1.27 1.27)
+				)
+				(hide yes)
+			)
+		)
+		(pin "1"
+		)
+		(instances
+			(project "CustomKeyboard"
+				(path "/e015e616-37c3-4f95-aa49-76389b12ce2e"
+					(reference "#PWR05")
+					(unit 1)
+				)
